File: osumgp-rp2040.kicad_pcb (KiCad board)
At the start: 2 copper layers, 130 x 51 mm, 92 parts, among them J1 USB_C_Receptacle_USB2.0, J2 SWD, J3 USB, J4 I2C, SW1 BOOTSEL, SW2 RST, SW3 Alpsalpine_RKJXV, SW4 Alpsalpine_RKJXV, U2 W25Q16JVUXIQ, U4 USBLC6-2P6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

Commit message: Fix DRC
Parts:
- moved C8 1.22 mm to (119.5, 58.0)
- moved C15 1.12 mm to (118.8, 57.3)
- moved C10 0.20 mm to (114.4, 58.0)
- moved C12 0.20 mm to (113.4, 58.0)
- moved R8 0.20 mm to (116.5, 58.0)
- moved R9 0.20 mm to (115.4, 58.0)
- moved C11 0.11 mm to (112.2, 65.2)
Connections:
- J3 pad MP: (no net) -> unconnected-(J3-PadMP)_0
- J4 pad MP: (no net) -> unconnected-(J4-PadMP)_0
Routing:
- net +3V3: track 207.7 -> 195.0 mm
- net /BUTTON_L3: track 60.5 -> 57.3 mm
- net +1V1: track 10.4 -> 8.70 mm
- net GND: track 5.50 -> 4.05 mm, vias 67 -> 68
