File: osumgp-rp2040.kicad_pcb (KiCad board)
At the start: 2 copper layers, 130 x 51 mm, 92 parts, among them J1 USB_C_Receptacle_USB2.0, J2 SWD, J3 USB, J4 I2C, SW1 BOOTSEL, SW2 RST, SW3 Alpsalpine_RKJXV, SW4 Alpsalpine_RKJXV, U2 W25Q16JVUXIQ, U4 USBLC6-2P6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

Commit message: beta 0.4
- copper to edge clearance 0.38mm
- fix thin +3.3V traces
- add more GND around the RP2040
- connected mounting pads to GND
- add more GND stitching
- reduce plane fingers
- reduce top/bottom traces running in parallel
Connections:
- J3 pad MP: (no net) -> GND
- J4 pad MP: (no net) -> GND
Routing:
- net /THUMBSTICK_LEFT_Y: track 76.4 -> 73.6 mm
- net /THUMBSTICK_RIGHT_Y: track 37.7 -> 40.4 mm
- net +3V3: track 207.7 -> 205.1 mm
- net /BUTTON_L3: track 60.5 -> 61.5 mm
- net /THUMBSTICK_RIGHT_X: track 52.1 -> 53.0 mm
- net /BUTTON_UP: track 28.1 -> 28.9 mm
- net GND: vias 67 -> 107
Other:
- board text added: "BETA 0.4"
- board text removed: "BETA 0.3"

Commit message: fix led
Parts:
- moved R2 5.73 mm to (106.5, 48.8)
- renumbered D2 to D1, R12 to R2
Connections:
- D1 pad 1: Net-(D2-K) -> GND
- D1 pad 2: /GPIO25 -> Net-(D1-A)
- J3 pad MP: GND -> (no net)
- J4 pad MP: GND -> (no net)
- R2 pad 1: Net-(D2-K) -> /GPIO25
- R2 pad 2: GND -> Net-(D1-A)
Routing:
- net /GPIO25: track 22.2 -> 19.2 mm
- net Net-(D1-A): track 0.00 -> 1.95 mm
- net Net-(D2-K): track 1.41 -> 0.00 mm
