File: osumgp-rp2040.kicad_sch (KiCad schematic)
At the start: 76 parts, among them J1 USB_C_Receptacle_USB2.0, J2 SWD, J3 USB, J4 I2C, SW1 BOOTSEL, SW2 RST, SW3 Alpsalpine_RKJXV, SW4 Alpsalpine_RKJXV, U2 W25Q16JVUXIQ, U4 USBLC6-2P6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

Commit message: Fix DRC
Connections:
- no-connect marks 4 -> 10
Other:
- moved on the sheet: S1, S10, S11, S12, S14, S2, S3, S4, S5, S6, S7, S8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
