File: osumgp-rp2040.kicad_sch (KiCad schematic)
At the start: 76 parts, among them J1 USB_C_Receptacle_USB2.0, J2 SWD, J3 USB, J4 I2C, SW1 BOOTSEL, SW2 RST, SW3 Alpsalpine_RKJXV, SW4 Alpsalpine_RKJXV, U2 W25Q16JVUXIQ, U4 USBLC6-2P6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

Commit message: beta 0.4
- copper to edge clearance 0.38mm
- fix thin +3.3V traces
- add more GND around the RP2040
- connected mounting pads to GND
- add more GND stitching
- reduce plane fingers
- reduce top/bottom traces running in parallel
Changed lines of the file:
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@@
 	)
 	(junction
-		(at 53.34 29.21)
-		(diameter 0)
-		(color 0 0 0 0)
-	)
-	(junction
 		(at 238.76 165.1)
 		(diameter 0)
@@
 	(wire
 		(pts
+			(xy 67.31 29.21) (xy 104.14 29.21)
+		)
+		(stroke
+			(width 0)
+			(type default)
+		)
+	)
+	(wire
+		(pts
 			(xy 110.49 31.75) (xy 111.76 31.75)
 		)
@@
 	(wire
 		(pts
-			(xy 53.34 29.21) (xy 67.31 29.21)
+			(xy 50.8 29.21) (xy 67.31 29.21)
 		)
 		(stroke
@@
 	(wire
 		(pts
-			(xy 50.8 29.21) (xy 53.34 29.21)
-		)
-		(stroke
-			(width 0)
-			(type default)
-		)
-	)
-	(wire
-		(pts
 			(xy 111.76 256.54) (xy 115.57 256.54)
 		)
@@
 	(wire
 		(pts
-			(xy 53.34 27.94) (xy 53.34 29.21)
-		)
-		(stroke
-			(width 0)
-			(type default)
-		)
-	)
-	(wire
-		(pts
 			(xy 124.46 146.685) (xy 127 146.685)
 		)
@@
 	(wire
 		(pts
-			(xy 67.31 29.21) (xy 104.14 29.21)
-		)
-		(stroke
-			(width 0)
-			(type default)
-		)
-	)
-	(wire
-		(pts
 			(xy 353.06 109.22) (xy 356.87 109.22)
 		)
@@
 			)
 		)
-		(property "Value" "VBUS"
+		(property "Value" "+5V"
 			(at 44.45 90.17 0)
 			(effects
@@
 					(unit 1)
 				)
-			)
-		)
-	)
-	(symbol
-		(lib_id "power:VBUS")
-		(at 53.34 27.94 0)
-		(unit 1)
-		(exclude_from_sim no)
-		(in_bom yes)
-		(on_board yes)
-		(dnp no)
-		(fields_autoplaced yes)
-		(property "Reference" "#PWR010"
-			(at 53.34 31.75 0)
-			(effects
-				(font
-					(size 1.27 1.27)
-				)
-				(hide yes)
-			)
-		)
-		(property "Value" "VBUS"
-			(at 53.34 22.225 0)
-			(effects
-				(font
-					(size 1.27 1.27)
-				)
-			)
-		)
-		(property "Footprint" ""
-			(at 53.34 27.94 0)
-			(effects
-				(font
-					(size 1.27 1.27)
-				)
-				(hide yes)
-			)
-		)
-		(property "Datasheet" ""
-			(at 53.34 27.94 0)
-			(effects
-				(font
-					(size 1.27 1.27)
-				)
-				(hide yes)
-			)
-		)
-		(property "Description" ""
-			(at 53.34 27.94 0)
-			(effects
-				(font
-					(size 1.27 1.27)
-				)
-				(hide yes)
-			)
-		)
-		(pin "1"
-		)
-		(instances
-			(project "osumgp-rp2040"
-				(path "/73e46140-01b8-4ec1-93bb-0d72bea0e0ee"
-					(reference "#PWR010")
-					(unit 1)
-				)

Commit message: fix led
Parts:
- removed D2: LED, LED_SMD:LED_0603_1608Metric_Pad1.05x0.95mm_HandSolder, symbol Device:LED
- removed R3: 1kΩ, Resistor_SMD:R_0402_1005Metric, symbol Device:R
- added D1: LED, LED_SMD:LED_0603_1608Metric_Pad1.05x0.95mm_HandSolder, symbol Device:LED
- added R2: 1kΩ, Resistor_SMD:R_0402_1005Metric, symbol Device:R
Connections:
- net GND: now also D1.1 (K)
- net GPIO25: now also R2.1
- new net: D1.2 (A), R2.2
